File: Eagle/LCD_v0_1/Bio_v4_LCD.brd (EAGLE design)
At the start: 69.2 x 40.4 mm, 39 parts, among them X2 16MHz, X3 FH12-08S-1SH, X4 MINI-USB

Commit message: Update value label position
Parts:
- 32U4: value ATMEGA32U4 -> 32U4
Other:
- board text added: "Screen v0.1"
- board text removed: "PID"
- board text removed: "Screen"
