File: Eagle/LCD_v0_2/Bio_v4_LCD0_2.brd (EAGLE design)
At the start: 69.2 x 40.4 mm, 39 parts, among them X2 16MHz, X3 FH12-08S-1SH, X4 MINI-USB

Commit message: swapped flex connector on LCD SPI, changed D11 pin by the SS/RXLED pin instead, removed SPI pull-up + diode
Parts:
- removed LDSLAVE: RED, adafruit:CHIP-LED0805
- removed RK18: 10k, rcl:R0805
- 32U4: value ATMEGA32U4 -> 32U4
- moved R1 5.32 mm to (15.0, 69.5)
- moved C13 2.56 mm to (19.2, 67.6)
- moved CU3 0.17 mm to (22.0, 70.5)
Connections:
- removed net N$22: LDSLAVE.A, RK18.2
- net +5V/1: now also X3.7, X3.8; no longer RK18.1, X3.1, X3.2
- net CS_32U4: now also X3.3; no longer LDSLAVE.C, X3.6
- net D11*: no longer R1.2
- net GND: now also X3.1, X3.2; no longer X3.7, X3.8
- net MISO: now also X3.4; no longer X3.5
- net MOSI: now also X3.5; no longer X3.4
- net RXLED: now also R1.2
- net SCK: now also X3.6; no longer X3.3
Routing:
- net SCK: track 26.9 -> 46.2 mm, vias 1 -> 3
- net CS_32U4: track 15.3 -> 6.05 mm
- net D11*: track 9.19 -> 0.00 mm
- net RXLED: track 0.00 -> 8.79 mm
- net N$1: track 2.55 -> 5.42 mm
- net N$22: track 2.08 -> 0.00 mm
- net GND: track 72.8 -> 70.7 mm
- net MISO: track 30.3 -> 28.4 mm, vias 1 -> 2
- net MOSI: track 29.2 -> 30.6 mm
- net +5V/1: track 214.3 -> 213.7 mm
Other:
- board text added: "Screen v0.1"
- board text removed: "PID"
- board text removed: "SPI"
- board text removed: "Screen"
