File: Eagle/LCD_v0_2/Bio_v4_LCD0_2.sch (EAGLE design)
At the start: 39 parts, among them X2 16MHz, X3 FH12-08S-1SH, X4 MINI-USB

Commit message: swapped flex connector on LCD SPI, changed D11 pin by the SS/RXLED pin instead, removed SPI pull-up + diode
Parts:
- removed LDSLAVE: RED, adafruit:LEDCHIP-LED0805
- removed RK18: 10k, rcl:R-EU_R0805
- 32U4: value ATMEGA32U4 -> 32U4
Connections:
- removed net N$22: LDSLAVE.A, RK18.2
- net +5V/1: now also X3-7.1, X3-8.1; no longer RK18.1, X3-1.1, X3-2.1
- net CS_32U4: now also X3-3.1; no longer LDSLAVE.C, X3-6.1
- net D11*: no longer R1.2
- net GND: now also X3-1.1, X3-2.1; no longer X3-7.1, X3-8.1
- net MISO: now also X3-4.1; no longer X3-5.1
- net MOSI: now also X3-5.1; no longer X3-4.1
- net RXLED: now also R1.2
- net SCK: now also X3-6.1; no longer X3-3.1
Changed lines of the file:
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@@
 <part name="GND21" library="supply1" deviceset="GND" device=""/>
 <part name="C10" library="rcl" deviceset="C-EU" device="C1206" value="100nF"/>
-<part name="32U4" library="adafruit" deviceset="ATMEGA32U4" device="-AU" value="ATMEGA32U4"/>
+<part name="32U4" library="adafruit" deviceset="ATMEGA32U4" device="-AU" value="32U4"/>
 <part name="CX2" library="rcl" deviceset="C-EU" device="C1206" value="22pF"/>
 <part name="CX1" library="rcl" deviceset="C-EU" device="C1206" value="22pF"/>
@@
 <part name="GND50" library="supply1" deviceset="GND" device=""/>
 <part name="C1" library="rcl" deviceset="C-EU" device="C1206" value="100nF"/>
-<part name="RK18" library="rcl" deviceset="R-EU_" device="R0805" value="10k"/>
-<part name="LDSLAVE" library="adafruit" deviceset="LED" device="CHIP-LED0805" value="RED"/>
-<part name="SUPPLY27" library="supply2" deviceset="+5V/1" device=""/>
 <part name="GND" library="Headerlibrary" deviceset="PINHD-1X1" device=""/>
 <part name="5V1" library="Headerlibrary" deviceset="PINHD-1X1" device=""/>
@@
 <instance part="X3" gate="-7" x="73.66" y="248.92"/>
 <instance part="X3" gate="-8" x="73.66" y="246.38"/>
-<instance part="GND6" gate="1" x="60.96" y="243.84"/>
-<instance part="SUPPLY4" gate="G$1" x="60.96" y="266.7"/>
+<instance part="GND6" gate="1" x="68.58" y="269.24" rot="R180"/>
+<instance part="SUPPLY4" gate="G$1" x="68.58" y="243.84" rot="R180"/>
 <instance part="R1" gate="G$1" x="55.88" y="243.84" rot="R270"/>
 <instance part="SJ1" gate="1" x="25.4" y="180.34" rot="R90"/>
@@
 <instance part="GND50" gate="1" x="165.1" y="256.54"/>
 <instance part="C1" gate="G$1" x="167.64" y="264.16"/>
-<instance part="RK18" gate="G$1" x="170.18" y="101.6" rot="MR270"/>
-<instance part="LDSLAVE" gate="G$1" x="170.18" y="88.9" rot="MR0"/>
-<instance part="SUPPLY27" gate="G$1" x="170.18" y="109.22"/>
 <instance part="GND" gate="G$1" x="22.86" y="114.3"/>
 <instance part="5V1" gate="G$1" x="22.86" y="104.14"/>
@@
 </segment>
 <segment>
-<pinref part="X3" gate="-8" pin="1"/>
-<wire x1="71.12" y1="246.38" x2="60.96" y2="246.38" width="0.1524" layer="91"/>
-<label x="60.96" y="246.38" size="1.778" layer="95"/>
-<pinref part="GND6" gate="1" pin="GND"/>
-<pinref part="X3" gate="-7" pin="1"/>
-<wire x1="71.12" y1="248.92" x2="60.96" y2="248.92" width="0.1524" layer="91"/>
-<label x="60.96" y="248.92" size="1.778" layer="95"/>
-<wire x1="60.96" y1="246.38" x2="60.96" y2="248.92" width="0.1524" layer="91"/>
-<junction x="60.96" y="246.38"/>
-</segment>
-<segment>
 <pinref part="32U4" gate="G$1" pin="GND2"/>
 <wire x1="86.36" y1="114.3" x2="83.82" y2="114.3" width="0.1524" layer="91"/>
@@
 <pinref part="GND8" gate="1" pin="GND"/>
 </segment>
+<segment>
+<pinref part="X3" gate="-2" pin="1"/>
+<pinref part="GND6" gate="1" pin="GND"/>
+<wire x1="71.12" y1="261.62" x2="68.58" y2="261.62" width="0.1524" layer="91"/>
+<wire x1="68.58" y1="261.62" x2="68.58" y2="264.16" width="0.1524" layer="91"/>
+<pinref part="X3" gate="-1" pin="1"/>
+<wire x1="68.58" y1="264.16" x2="68.58" y2="266.7" width="0.1524" layer="91"/>
+<wire x1="71.12" y1="264.16" x2="68.58" y2="264.16" width="0.1524" layer="91"/>
+<junction x="68.58" y="264.16"/>
+</segment>
 </net>
 <net name="SCK" class="0">
@@
 </segment>
 <segment>
-<pinref part="X3" gate="-3" pin="1"/>
-<wire x1="71.12" y1="259.08" x2="60.96" y2="259.08" width="0.1524" layer="91"/>
-<label x="60.96" y="259.08" size="1.778" layer="95"/>
+<pinref part="X3" gate="-6" pin="1"/>
+<wire x1="71.12" y1="251.46" x2="60.96" y2="251.46" width="0.1524" layer="91"/>
+<label x="60.96" y="251.46" size="1.778" layer="95"/>
 </segment>
 </net>
@@
 </segment>
 <segment>
+<pinref part="X3" gate="-4" pin="1"/>
+<wire x1="71.12" y1="256.54" x2="60.96" y2="256.54" width="0.1524" layer="91"/>
+<label x="60.96" y="256.54" size="1.778" layer="95"/>
+</segment>
+</net>
+<net name="MOSI" class="0">
+<segment>
+<pinref part="CON_ISP" gate="G$1" pin="MOSI"/>
+<wire x1="127" y1="254" x2="134.62" y2="254" width="0.1524" layer="91"/>
+<label x="132.08" y="254" size="1.778" layer="95"/>
+</segment>
+<segment>
+<pinref part="32U4" gate="G$1" pin="PB2(PDI/MOSI)"/>
+<wire x1="134.62" y1="139.7" x2="149.86" y2="139.7" width="0.1524" layer="91"/>
+<label x="144.78" y="139.7" size="1.778" layer="95"/>
+</segment>
+<segment>
 <pinref part="X3" gate="-5" pin="1"/>
 <wire x1="71.12" y1="254" x2="60.96" y2="254" width="0.1524" layer="91"/>
@@
 </segment>
 </net>
-<net name="MOSI" class="0">
-<segment>
-<pinref part="CON_ISP" gate="G$1" pin="MOSI"/>
-<wire x1="127" y1="254" x2="134.62" y2="254" width="0.1524" layer="91"/>
-<label x="132.08" y="254" size="1.778" layer="95"/>
-</segment>
-<segment>
-<pinref part="32U4" gate="G$1" pin="PB2(PDI/MOSI)"/>
-<wire x1="134.62" y1="139.7" x2="149.86" y2="139.7" width="0.1524" layer="91"/>
-<label x="144.78" y="139.7" size="1.778" layer="95"/>
-</segment>
-<segment>
-<pinref part="X3" gate="-4" pin="1"/>
-<wire x1="71.12" y1="256.54" x2="60.96" y2="256.54" width="0.1524" layer="91"/>
-<label x="60.96" y="256.54" size="1.778" layer="95"/>
-</segment>
-</net>
 <net name="USB_N" class="0">
 <segment>
@@
 <wire x1="134.62" y1="152.4" x2="149.86" y2="152.4" width="0.1524" layer="91"/>
 <label x="144.78" y="152.4" size="1.778" layer="95"/>
-</segment>
-<segment>
-<pinref part="R1" gate="G$1" pin="2"/>
-<wire x1="55.88" y1="238.76" x2="76.2" y2="238.76" width="0.1524" layer="91"/>
-<label x="68.58" y="238.76" size="1.778" layer="95"/>
 </segment>
 </net>
@@
 <wire x1="134.62" y1="134.62" x2="149.86" y2="134.62" width="0.1524" layer="91"/>
 <label x="144.78" y="134.62" size="1.778" layer="95"/>
+</segment>
+<segment>
+<pinref part="R1" gate="G$1" pin="2"/>
+<wire x1="55.88" y1="238.76" x2="55.88" y2="231.14" width="0.1524" layer="91"/>
+<label x="58.42" y="233.68" size="1.778" layer="95"/>
 </segment>
 </net>
@@
 </segment>
 <segment>
-<pinref part="X3" gate="-1" pin="1"/>
-<wire x1="71.12" y1="264.16" x2="60.96" y2="264.16" width="0.1524" layer="91"/>
-<label x="60.96" y="264.16" size="1.778" layer="95"/>
-<pinref part="SUPPLY4" gate="G$1" pin="+5V/1"/>
-<pinref part="X3" gate="-2" pin="1"/>
-<wire x1="71.12" y1="261.62" x2="60.96" y2="261.62" width="0.1524" layer="91"/>
-<label x="60.96" y="261.62" size="1.778" layer="95"/>
-<wire x1="60.96" y1="264.16" x2="60.96" y2="261.62" width="0.1524" layer="91"/>
-<junction x="60.96" y="264.16"/>
-</segment>
-<segment>
 <pinref part="32U4" gate="G$1" pin="AVCC"/>
 <wire x1="86.36" y1="165.1" x2="76.2" y2="165.1" width="0.1524" layer="91"/>
@@
 </segment>
 <segment>
-<pinref part="RK18" gate="G$1" pin="1"/>
-<pinref part="SUPPLY27" gate="G$1" pin="+5V/1"/>
-</segment>
-<segment>
 <pinref part="5V1" gate="G$1" pin="1"/>
 <pinref part="SUPPLY31" gate="G$1" pin="+5V/1"/>
@@
 <pinref part="RK2" gate="G$1" pin="2"/>
 <pinref part="SUPPLY10" gate="G$1" pin="+5V/1"/>
+</segment>
+<segment>
+<pinref part="X3" gate="-8" pin="1"/>
+<pinref part="SUPPLY4" gate="G$1" pin="+5V/1"/>
+<wire x1="71.12" y1="246.38" x2="68.58" y2="246.38" width="0.1524" layer="91"/>
+<pinref part="X3" gate="-7" pin="1"/>
+<wire x1="71.12" y1="248.92" x2="68.58" y2="248.92" width="0.1524" layer="91"/>
+<wire x1="68.58" y1="248.92" x2="68.58" y2="246.38" width="0.1524" layer="91"/>
+<junction x="68.58" y="246.38"/>
 </segment>
 </net>
@@
 <net name="CS_32U4" class="0">
 <segment>
-<pinref part="X3" gate="-6" pin="1"/>
-<wire x1="71.12" y1="251.46" x2="55.88" y2="251.46" width="0.1524" layer="91"/>
 <pinref part="R1" gate="G$1" pin="1"/>
-<wire x1="55.88" y1="251.46" x2="55.88" y2="248.92" width="0.1524" layer="91"/>
-<label x="60.96" y="251.46" size="1.778" layer="95"/>
-</segment>
-<segment>
-<pinref part="LDSLAVE" gate="G$1" pin="C"/>
-<wire x1="170.18" y1="83.82" x2="170.18" y2="73.66" width="0.1524" layer="91"/>
-<label x="170.18" y="73.66" size="1.778" layer="95" rot="R90"/>
+<label x="60.96" y="259.08" size="1.778" layer="95"/>
+<pinref part="X3" gate="-3" pin="1"/>
+<wire x1="71.12" y1="259.08" x2="55.88" y2="259.08" width="0.1524" layer="91"/>
+<wire x1="55.88" y1="259.08" x2="55.88" y2="248.92" width="0.1524" layer="91"/>
 </segment>
 </net>
@@
 </segment>
 </net>
-<net name="N$22" class="0">
-<segment>
-<pinref part="RK18" gate="G$1" pin="2"/>
-<wire x1="170.18" y1="91.44" x2="170.18" y2="96.52" width="0.1524" layer="91"/>
-<pinref part="LDSLAVE" gate="G$1" pin="A"/>
-</segment>
-</net>
