File: Eagle/Bertha_4_2/Bertha_v4_2.sch (EAGLE design)
At the start: 124 parts, among them CON1 JACK_DC_BARREL, IC1 MCP1703DB, IC3 SN74LVC2G14, J1 RJ12RIGHTANGLE-I2C, J2 RJ12RIGHTANGLE-I2C, J7 22--02, Q1 BSP75, Q2 BSP75, Q3 BSP75, Q4 BSP75, Q5 BSP75, Q6 BSP75, U1 HX711, U100 RN2483, X2 16MHz, X3 FH12-08S-1SH, X4 MINI-USB

Commit message: bioreactor v4.2 revision, Lora Reset pin on D5, operation at 8MHz, 3.3V. The Flex cable is now exporting 12V instead of 5V (careful, not compatible with LCD V0.2 sudo git add --all), I2C ports are only providing 12V
Parts:
- removed 5V1: (no value), Headerlibrary:PINHD-1X1
- removed CU5, CU6: 10uF, rcl:C-EUC1206
- removed D3: 1N581D1206, lpatiny:1N581D1206
- removed LDPW5: RED, adafruit:LEDCHIP-LED0805
- removed R13: 1k, resistor:R-EU_R0805
- removed U$2: NCP1117LPST50T3G, lpatiny:NCP1117LPST50T3G
Connections:
- removed net +5V: CU5.1, D3.A, U$2.OUT, U$2.TAB_OUT
- removed net +5V/1: 32U4.AVCC, 32U4.AVCC1, 32U4.UVCC, 32U4.VCC, 32U4.VCC1, 5V1.1, BJ1.E, C1.1, C12.2, C2.1, C6.1, CU1.1, CU3.1, CU4.1, CU7.1, D2.C, D3.C, D4.C, IC1.VI, IC3P.VCC, J1.5, J2.5, R13.1, R4.2, RK1.1, RK15.1, RK16.1, RK18.1, RK19.1, RK2.1, RK5.2, RK6.2, RT1.1, RT2.1, U$4.VDD, U$8.VCC, U1.DVDD, U1.VSUP, X3-1.1, X3-2.1
- removed net LORA_RST: 100K.2, LORA_RST.1, U100.P$32
- removed net N$12: LDPW5.A, R13.2
- removed net RX3: U100.P$6
- removed net TX3: U100.P$7
- net +12V: now also C1.1, C2.1, CU3.1, CU4.1, CU7.1, D2.C, D4.C, IC1.VI, X3-1.1, X3-2.1; no longer CU6.1, U$2.IN
- net 3.3V: now also 32U4.AVCC, 32U4.AVCC1, 32U4.UVCC, 32U4.VCC, 32U4.VCC1, BJ1.E, C12.2, C6.1, CU1.1, IC3P.VCC, R4.2, RK1.1, RK15.1, RK16.1, RK18.1, RK19.1, RK2.1, RK5.2, RK6.2, RT1.1, RT2.1, U$4.VDD, U$8.VCC, U1.DVDD, U1.VSUP
- net D5*: now also 100K.2, LORA_RST.1, U100.P$32
- net GND: no longer CU5.2, CU6.2, LDPW5.C, U$2.ADJ
- net RX: now also U100.P$6
- net TX: now also U100.P$7
Other:
- note removed: "5V LDO"
