File: Eagle/LCD_v1_0/Bio_v4_LCD1_0.sch (EAGLE design)
At the start: 117 parts, among them CON1 JACK_DC_BARREL, IC1 MCP1703DB, IC3 SN74LVC2G14, J1 RJ12RIGHTANGLE-I2C, J2 RJ12RIGHTANGLE-I2C, J7 22--02, Q1 BSP75, Q2 BSP75, Q3 BSP75, Q4 BSP75, Q5 BSP75, Q6 BSP75, U1 HX711, U100 RN2483, X2 8MHz, X3 FH12-08S-1SH, X4 MINI-USB

Commit message: LCD v1_0, compatible with v4_2 of the main board, 5V generated on board w NCP1117
Parts:
- removed 100K: 100k, rcl:R-EU_R0805
- removed 12V, 3V3, AN_OUT, LORA_RST: (no value), Headerlibrary:PINHD-1X1
- removed 20K: 20k, resistor:R-EU_M0805
- removed 8.2K: 8.2k, resistor:R-EU_M0805
- removed BJ1: MMBT4403, SparkFun-DiscreteSemi:TRANSISTOR_PNPMMBT4403
- removed C2, C3, C4, C5, C6, C7, C8, C9: 100nF, rcl:C-EUC1206
- removed CON1: JACK_DC_BARREL, lpatiny:JACK_DC_BARREL
- removed CU1, CU2, CU4, CU7, CU8: 10uF, rcl:C-EUC1206
- removed HX1: IRF3704S, transistor-power:IRF3704S
- removed IC1: MCP1703DB, linear:MCP1703DB
- removed IC3: SN74LVC2G14, lpatiny:SN74LVC2G14
- removed IN, OUT: (no value), jumper:JP1E
- removed J1, J2: RJ12RIGHTANGLE-I2C, lpatiny:RJ12RIGHTANGLE-I2C
- removed J7: 22--02, lpatiny:22--02
- removed JP2: M02PTH, SparkFun-Connectors:M02PTH
- removed LDIN, LDM1, LDM2, LDM3, LDM4, LDMEM, LDOUT, LDPID, LDPW12, LDPW3, LDSLAVE, RXLD, TXLD: RED, adafruit:LEDCHIP-LED0805
- removed Q1, Q2, Q3, Q4, Q5, Q6: BSP75, infineon:BSP613P
- removed R10, R11, R4, R5, R6, R9: 1K, rcl:R-EU_R0805
- removed R12: 1k, rcl:R-EU_R0805
- removed R14: 1k, resistor:R-EU_R0805
- removed RK10, RK11, RK8, RK9: 10K, rcl:R-EU_R0805
- removed RK12, RK13, RK14, RK15, RK16, RK18, RK19, RK3, RK4: 10k, rcl:R-EU_R0805
- removed RK5: 10k, resistor:R-EU_M0805
- removed RL1, RL2: 100, resistor:R-EU_M0805
- removed RT1, RT2: 4.7k, resistor:R-EU_R1206
- removed SJ2, SJ4, SJ5, SJ6: JUMPER-PAD-2-NC_BY_TRACE, SparkFun-Passives:JUMPER-PAD-2-NC_BY_TRACE
- removed SJ3: (no value), jumper:SJ
- removed STEPPER: (no value), con-lsta:FE06-1
- removed U$4: DS18B20, lpatiny:DS18B20
- removed U$8: DS18B20_SMALLPADS, lpatiny:DS18B20_SMALLPADS
- removed U1: HX711, Testing:HX711HX711
- removed U100: RN2483, Octanis1:RN2483
- removed WGT: (no value), SparkFun-Connectors:M05PTH
- added 220: 220, rcl:R-EU_R0805
- added 5V1: (no value), Headerlibrary:PINHD-1X1
- added CU5, CU6: 10uF, rcl:C-EUC1206
- added LCD: (no value), lpatiny:LCD-HEADER
- added LDO: NCP1117LPST50T3G, lpatiny:NCP1117LPST50T3G
- added LDPW5: RED, adafruit:LEDCHIP-LED0805
- added R13: 1k, resistor:R-EU_R0805
- added RE1, RE2: 5k, rcl:R-EU_R0805
- 32U4: value ATMEGA32U4 -> 32U4
- R2: value 10k -> 1k
- RK1: value 10K -> 10k; device resistor:R-EU_M0805 -> rcl:R-EU_R0805
- RK2: value 10K -> 10k
- U$1: value SST25VF064C -> EC11E; device BertaLib:SST25VF064C -> lpatiny:EC11E
- X2: value 8MHz -> 16MHz
Connections:
- removed net 3.3V: 100K.1, 32U4.AVCC, 32U4.AVCC1, 32U4.UVCC, 32U4.VCC, 32U4.VCC1, 3V3.1, BJ1.E, C12.2, C3.1, C4.1, C5.2, C6.1, CU1.1, CU8.1, IC1.VO, IC3P.VCC, R14.1, R4.2, RK1.1, RK15.1, RK16.1, RK18.1, RK19.1, RK2.1, RK4.2, RK5.2, RK6.2, RT1.1, RT2.1, U$1.HOLD, U$1.VCC, U$1.WP, U$4.VDD, U$8.VCC, U1.DVDD, U1.VSUP, U100.P$12, U100.P$34
- removed net A+: RL2.2, WGT.2
- removed net A-: RL1.2, WGT.3
- removed net ANGND: C3.2, C4.2, SJ4.2, SJ5.2, SJ6.2, U100.P$1, U100.P$11, U100.P$20, U100.P$21, U100.P$22, U100.P$24, U100.P$26, U100.P$27, U100.P$28, U100.P$33, U100.P$41, U100.P$47, U100.P$8
- removed net ANT868: AN_OUT.1, U100.P$23
- removed net B+: JP2.1, U1.INB+
- removed net B-: JP2.2, U1.INB-
- removed net CN3: C8.2, U1.VBG
- removed net LGND: 8.2K.1, C7.2, C8.1, CU2.2, SJ2.2, U1.AGND
- removed net N$10: R3.1, U$1.CS
- removed net N$13: OUT.2, Q5.D@1
- removed net N$14: Q4.D@1, RK8.1, STEPPER.1
- removed net N$15: Q2.D@1, RK9.1, STEPPER.3
- removed net N$16: Q3.D@1, RK10.1, STEPPER.4
- removed net N$17: IN.2, Q6.D@1
- removed net N$18: RK15.2, TXLD.A
- removed net N$19: Q1.D@1, RK11.1, STEPPER.6
- removed net N$20: C9.2, RL1.1, U1.INA-
- removed net N$21: R9.2, RT1.2, U$8.DQ
- removed net N$22: LDSLAVE.A, RK18.2
- removed net N$23: RK3.2, U$1.SCK
- removed net N$24: RK16.2, RXLD.A
- removed net N$25: LDMEM.A, RK19.2
- removed net N$26: LDPID.A, RK14.1
- removed net N$27: LDIN.A, RK12.1
- removed net N$28: LDOUT.A, RK13.1
- removed net N$29: IC3A.O, Q3.G
- removed net N$30: IC3B.O, Q1.G
- removed net N$31: LDM4.C, RK8.2
- removed net N$32: LDM3.C, RK9.2
- removed net N$33: LDM2.C, RK10.2
- removed net N$34: LDPW3.A, R14.2
- removed net N$36: HX1.D, J7-2.S
- removed net N$37: LDM1.C, RK11.2
- removed net N$38: BJ1.B, U1.BASE
- removed net N$39: 20K.1, 8.2K.2, U1.VFB
- removed net N$41: RK5.1, SJ3.1, U1.RATE
- removed net N$43: C9.1, RL2.1, U1.INA+
- removed net N$5: 20K.2, BJ1.C, C7.1, CU2.1, U1.AVDD, WGT.5
- removed net N$6: HX1.G, R11.2, RK14.2
- removed net N$7: LDPW12.A, R12.1
- removed net N$8: Q6.G, R5.2, RK12.2
- removed net N$9: R10.2, RT2.2, U$4.DQ
- new net +5V/1: 220.1, 32U4.AVCC, 32U4.AVCC1, 32U4.UVCC, 32U4.VCC, 32U4.VCC1, 5V1.1, C1.1, C12.2, CU3.1, CU5.1, D2.C, D4.C, LCD.2, LDO.OUT, LDO.TAB_OUT, R13.1, RE1.1, RE2.1, RK1.1, RK2.2, RK6.2
- new net N$12: LDPW5.A, R13.2
- new net N$2: LCD.3, R3.1, RK1.2
- net +12V: now also CU6.1, LDO.IN, X3-7.1, X3-8.1; no longer 12V.1, C1.1, C2.1, CON1.V+, CU3.1, CU4.1, CU7.1, D2.C, D4.C, IC1.VI, IN.1, J1.1, J2.1, J7-1.S, LDM1.A, LDM2.A, LDM3.A, LDM4.A, OUT.1, R12.2, STEPPER.2, STEPPER.5, X3-1.1, X3-2.1
- net A0: no longer IC3B.I, Q2.G, R4.1
- net A1: no longer IC3A.I, Q4.G
- net A2: no longer R5.1
- net A3: no longer R6.1
- net A4: no longer U1.DOUT
- net A5: no longer U1.PD_SCK
- net A6: now also LCD.14; no longer R9.1
- net CS_32U4: now also X3-3.1; no longer LDSLAVE.C, X3-6.1
- net D10*: now also LCD.4; no longer LDMEM.C, R3.2
- net D11*: no longer R1.2
- net D12*: now also LCD.13; no longer R11.1
- net D5*: no longer 100K.2, LORA_RST.1, U100.P$32
- net D6*: now also LCD.12; no longer R10.1
- net D7*: now also RK2.1, U$1.INT
- net D8*: now also LCD.11
- net D9*: now also LCD.6
- net GND: now also CU5.2, CU6.2, LCD.1, LCD.16, LCD.5, LDO.ADJ, LDPW5.C, R3.2, U$1.CLSD, X3-1.1, X3-2.1; no longer C2.2, C5.1, C6.2, CON1.GND, CU1.2, CU4.2, CU7.2, CU8.2, HX1.S, IC1.GND, IC3P.GND, J1.4, J1.6, J2.4, J2.6, LDIN.C, LDOUT.C, LDPID.C, LDPW12.C, LDPW3.C, Q1.S, Q2.S, Q3.S, Q4.S, Q5.S, Q6.S, SJ2.1, SJ3.2, SJ4.1, SJ5.1, SJ6.1, U$4.GND, U$8.GND, U1.XI, WGT.1, WGT.4, X3-7.1, X3-8.1
- net MISO: now also X3-4.1; no longer U$1.MISO, X3-5.1
- net MOSI: now also X3-5.1; no longer RK4.1, U$1.MOSI, X3-4.1
- net N$11: now also 220.2, LCD.15; no longer Q5.G, R6.2, RK13.2
- net RX: now also RE2.2, U$1.B; no longer U100.P$6
- net RXLED: now also R1.2; no longer RXLD.C
- net SCK: now also X3-6.1; no longer RK3.1, X3-3.1
- net SCL: no longer J1.2, J2.2, RK2.2
- net SDA: no longer J1.3, J2.3, RK1.2
- net TX: now also RE1.2, U$1.A; no longer U100.P$7
- net TXLED: no longer TXLD.C
Other:
- note added: "5V LDO"
- note added: "LCD 20X4"
- note added: "Rot encoder"
- note removed: "3.3V LDO"
- note removed: "A+"
- note removed: "A-"
- note removed: "AVDD = VBG(R1+R2)/R1"
- note removed: "Black"
- note removed: "Default: Closed - Data rate set to 10SPS"
- note removed: "E+"
- note removed: "E-"
- note removed: "FOOD"
- note removed: "Flash Memory"
- note removed: "I2C"
- note removed: "IO: 2.7-5.5V"
- note removed: "LEVEL_Converters"
- note removed: "LoRa RN2483"
- note removed: "Load cell 24bits ADC"
- note removed: "One wire"
- note removed: "Open jumper to set to 80SPS Increases noise per read"
- note removed: "PID"
- note removed: "POWER_LEDS"
- note removed: "Power Supply"
- note removed: "Red"
- note removed: "STEPPER"
- note removed: "Shield"
- note removed: "VBG = 1.25V"
- note removed: "VCC: 2.7-5.5V"
- note removed: "White"
- note removed: "Yellow"
- moved on the sheet: 32U4, BKLD, C10, C11, C12, C13, CU9, CX1, CX2, D4, GND, R2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
