File: Eagle/pH_v5_0/ph_v5.sch (EAGLE design)
At the start: 142 parts, among them CON1 JACK_DC_BARREL, IC1 MCP1703DB, IC2 TL084D, IC3 TL084D, IC5 TPS60400DBV, J1 RJ12RIGHTANGLE-I2C, J2 RJ12RIGHTANGLE-I2C, Q1 BSP75, Q2 BSP75, Q3 BSP75, Q4 BSP75, Q5 BSP75, Q6 BSP75, Q7 BSP75, Q8 BSP75, U1 HX711, U100 RN2483, X2 8MHz, X3 FH12-08S-1SH, X4 MINI-USB

Commit message: Added SMA LoRa antenna for phV5 board extra mistakes fixed with DRC close #18
Parts:
- removed AN_OUT: (no value), Headerlibrary:PINHD-1X1
- added 868MHZ: (no value), sma_end_launch:SMACONNECTOR_EDGE
Connections:
- net ANGND: now also 868MHZ.GND1, 868MHZ.GND2, 868MHZ.GND3, 868MHZ.GND4
- net ANT868: now also 868MHZ.ANT; no longer AN_OUT.1
Changed lines of the file:
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@@
 <?xml version="1.0" encoding="utf-8"?>
 <!DOCTYPE eagle SYSTEM "eagle.dtd">
-<eagle version="6.5.0">
+<eagle version="7.6.0">
 <drawing>
 <settings>
@@
 <part name="P+25" library="SparkFun" deviceset="3.3V" device=""/>
 <part name="P+26" library="SparkFun" deviceset="3.3V" device=""/>
-<part name="AN_OUT" library="Headerlibrary" deviceset="PINHD-1X1" device=""/>
 <part name="RXT" library="rcl" deviceset="R-EU_" device="R0805" value="1M"/>
 <part name="C2" library="rcl" deviceset="C-EU" device="C1206" value="100nF"/>
@@
 <part name="GND30" library="supply1" deviceset="GND" device=""/>
 <part name="P+45" library="SparkFun" deviceset="3.3V" device=""/>
-<part name="SUPPLY5" library="supply2" deviceset="VSS" device=""/>
 <part name="B1" library="rectifier" deviceset="MB*S" device="" technology="1"/>
 <part name="C24" library="SparkysWidgets" deviceset="CAP" device="1206" value="100nF"/>
@@
 <part name="RK15" library="rcl" deviceset="R-EU_" device="R0805" value="10k"/>
 <part name="P+46" library="SparkFun" deviceset="3.3V" device=""/>
+<part name="868MHZ" library="sma_end_launch" deviceset="SMACONNECTOR" device="_EDGE"/>
 </parts>
 <sheets>
@@
 <instance part="P+25" gate="G$1" x="289.56" y="281.94"/>
 <instance part="P+26" gate="G$1" x="226.06" y="233.68" rot="R270"/>
-<instance part="AN_OUT" gate="G$1" x="274.32" y="254"/>
 <instance part="RXT" gate="G$1" x="271.78" y="132.08" rot="MR90"/>
 <instance part="C2" gate="G$1" x="167.64" y="241.3"/>
@@
 <instance part="GND30" gate="1" x="38.1" y="38.1" rot="R90"/>
 <instance part="P+45" gate="G$1" x="-2.54" y="43.18" rot="R90"/>
-<instance part="SUPPLY5" gate="G$1" x="55.88" y="48.26"/>
 <instance part="B1" gate="G$1" x="116.84" y="99.06" rot="R90"/>
 <instance part="C24" gate="G$1" x="86.36" y="114.3" smashed="yes" rot="R90">
@@
 <instance part="RK15" gate="G$1" x="398.78" y="40.64" rot="MR270"/>
 <instance part="P+46" gate="G$1" x="398.78" y="45.72"/>
+<instance part="868MHZ" gate="G$1" x="287.02" y="256.54"/>
 </instances>
 <busses>
@@
 <wire x1="271.78" y1="254" x2="243.84" y2="254" width="0.1524" layer="91"/>
 <label x="254" y="254" size="1.778" layer="95"/>
-<pinref part="AN_OUT" gate="G$1" pin="1"/>
+<pinref part="868MHZ" gate="G$1" pin="ANT"/>
+<wire x1="279.4" y1="256.54" x2="271.78" y2="256.54" width="0.1524" layer="91"/>
+<wire x1="271.78" y1="256.54" x2="271.78" y2="254" width="0.1524" layer="91"/>
 </segment>
 </net>
@@
 </segment>
 <segment>
+<wire x1="281.94" y1="269.24" x2="281.94" y2="271.78" width="0.1524" layer="91"/>
+<pinref part="C3" gate="G$1" pin="2"/>
+<wire x1="289.56" y1="271.78" x2="289.56" y2="269.24" width="0.1524" layer="91"/>
+<pinref part="C4" gate="G$1" pin="2"/>
+<wire x1="281.94" y1="269.24" x2="289.56" y2="269.24" width="0.1524" layer="91"/>
+<label x="281.94" y="266.7" size="1.778" layer="95"/>
+</segment>
+<segment>
+<pinref part="868MHZ" gate="G$1" pin="GND4"/>
+<pinref part="868MHZ" gate="G$1" pin="GND3"/>
+<wire x1="289.56" y1="248.92" x2="284.48" y2="248.92" width="0.1524" layer="91"/>
+<wire x1="284.48" y1="248.92" x2="248.92" y2="248.92" width="0.1524" layer="91"/>
+<junction x="284.48" y="248.92"/>
+<pinref part="868MHZ" gate="G$1" pin="GND2"/>
+<pinref part="868MHZ" gate="G$1" pin="GND1"/>
+<wire x1="289.56" y1="264.16" x2="284.48" y2="264.16" width="0.1524" layer="91"/>
+<wire x1="284.48" y1="264.16" x2="266.7" y2="264.16" width="0.1524" layer="91"/>
+<junction x="284.48" y="264.16"/>
 <pinref part="U100" gate="G$1" pin="P$27"/>
 <wire x1="243.84" y1="264.16" x2="248.92" y2="264.16" width="0.1524" layer="91"/>
@@
 <pinref part="SJ6" gate="G$1" pin="2"/>
 <junction x="248.92" y="259.08"/>
-</segment>
-<segment>
-<wire x1="281.94" y1="269.24" x2="281.94" y2="271.78" width="0.1524" layer="91"/>
-<pinref part="C3" gate="G$1" pin="2"/>
-<wire x1="289.56" y1="271.78" x2="289.56" y2="269.24" width="0.1524" layer="91"/>
-<pinref part="C4" gate="G$1" pin="2"/>
-<wire x1="281.94" y1="269.24" x2="289.56" y2="269.24" width="0.1524" layer="91"/>
-<label x="281.94" y="266.7" size="1.778" layer="95"/>
+<junction x="248.92" y="248.92"/>
+<wire x1="266.7" y1="264.16" x2="266.7" y2="269.24" width="0.1524" layer="91"/>
+<wire x1="266.7" y1="269.24" x2="248.92" y2="269.24" width="0.1524" layer="91"/>
+<wire x1="248.92" y1="269.24" x2="248.92" y2="264.16" width="0.1524" layer="91"/>
+<junction x="248.92" y="264.16"/>
 </segment>
 </net>
@@
 <pinref part="R20" gate="G$1" pin="2"/>
 <pinref part="IC3" gate="C" pin="+IN"/>
-<junction x="104.14" y="114.3"/>
 <pinref part="IC3" gate="C" pin="+IN"/>
 <wire x1="104.14" y1="114.3" x2="91.44" y2="114.3" width="0.1524" layer="91"/>
