File: Eagle/ph_v6_0/ph_v6.sch (EAGLE design)
At the start: 177 parts, among them CON1 JACK_DC_BARREL, IC1 MCP1703DB, IC2 TL084D, IC3 TL084D, IC4 DRV8811, IC5 TPS60400DBV, IC6 DRV8811, J1 RJ12RIGHTANGLE-I2C, J2 RJ12RIGHTANGLE-I2C, U1 HX711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

Commit message: Progress on pH board v6_0 with DRV8811
Parts:
- 20K, 8.2K, RK5: device resistor:R-EU_M0805 -> resistor:R-EU_R0805
- C1, C10, C11, C12, C13, C14, C15, C16, C2, C3, C4, C5, C6, C7, C8, CU1, CU2, CU3, CU4, CU7, CU8, CU9, CX1, CX2: device rcl:C-EUC1206 -> rcl:C-EUC0805
- C17, C18, C19, C20, C21, C22, C23, C24, C9: device SparkysWidgets:CAP1206 -> SparkysWidgets:CAP0805
- C25, C26, C27, C28, C29, C31, C32, C36, C37, C38, C39, C40, C42, C43, C44, C45, C46: device freetronics-master-v1:CAP0603 -> freetronics-master-v1:CAP0805
- C33: value 100nF 0603 -> 100nF; device freetronics-master-v1:CAP0603 -> freetronics-master-v1:CAP0805
- C34, C35: value 220nF 0603 -> 220nF; device freetronics-master-v1:CAP0603 -> freetronics-master-v1:CAP0805
- R25: value 3K3 -> 47K; device freetronics-master-v1:RESISTOR0603 -> freetronics-master-v1:RESISTOR0805
- R26: value 47K -> 0.2R 1W; device freetronics-master-v1:RESISTOR0603 -> rcl:R-EU_R2010
- R27, R28, R37, R39, R40, R41, R42, R43, R44, R45, R47, R48, R49, R50, R51: device freetronics-master-v1:RESISTOR0603 -> freetronics-master-v1:RESISTOR0805
- R29: value 10K -> 3k3; device freetronics-master-v1:RESISTOR0603 -> freetronics-master-v1:RESISTOR0805
- R30, R31, R33, R34, R35, R36: value 10K -> 10k; device freetronics-master-v1:RESISTOR0603 -> freetronics-master-v1:RESISTOR0805
- R32: value 0.2R 1W -> 10k; device rcl:R-EU_R2010 -> freetronics-master-v1:RESISTOR0805
Connections:
- removed net D2: IC4.DIR
- removed net D5: IC4.STEP
- removed net N$62: C30.1, IC4.ISENB, R32.2
- removed net N$63: C28.1, IC4.DECAY, R29.1, R37.2
- removed net N$64: C25.1, IC4.RCA, R26.2
- removed net N$68: C27.1, IC4.VREF, R25.1, R28.2
- removed net N$70: IC4.USM1, R30.1, SJ5.2
- removed net N$71: IC4.USM0, R31.1, SJ7.2
- new net N$13: C30.1, IC4.ISENB, R26.2
- new net N$14: C28.1, IC4.DECAY, R30.1, R37.2
- new net N$15: C25.1, IC4.RCA, R25.2
- new net N$32: C27.1, IC4.VREF, R28.2, R29.1
- new net N$37: IC4.USM1, R31.1, SJ5.2
- new net N$53: IC4.USM0, R32.1, SJ7.2
- net +12V: no longer X3-1.1, X3-2.1
- net 3.3V: now also R32.2; no longer R25.2
- net D3: now also IC4.DIR
- net D6: now also IC4.STEP
- net GND: now also R25.1; no longer R32.1
- net VDD: now also X3-1.1, X3-2.1
Other:
- note removed: "C13: 399-6104-ND"
- note removed: "CSRN2010FKR200CT-ND"
- note removed: "S1_DIR"
- note removed: "S1_STEP"
- note removed: "Stepper 1"
- moved on the sheet: C25, C26, C27, C28, C29, C30, C31, C32, C33, C34, C35, C47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

Commit message: progress on phv6, mem select now on A3, LoRa reset on A1, Stepper 1(PWM D9, dir D8), Stepper 2(PWM D10, dir D5)
Parts:
- removed JP2: (no value), freetronics-master-v1:M04SCREW
- added JP3: (no value), jumper:JP4E
- JP1: device freetronics-master-v1:M04SCREW -> jumper:JP4E
Connections:
- removed net D3: IC4.DIR, IC6.DIR
- removed net D6: IC4.STEP, IC6.STEP
- net A1: now also 100K.2, LORA_RST.1, U100.P$32
- net A3: now also LDMEM.C, R3.2
- net D10*: now also IC6.STEP; no longer LDMEM.C, R3.2
- net D5*: now also IC6.DIR; no longer 100K.2, LORA_RST.1, U100.P$32
- net D8*: now also IC4.DIR
- net D9*: now also IC4.STEP
- net N$2: now also JP1.4; no longer JP1.1
- net N$4: now also JP1.2; no longer JP1.3
- net N$55: now also JP1.1; no longer JP1.4
- net N$56: now also JP1.3; no longer JP1.2
- net N$73: now also JP3.4; no longer JP2.1
- net N$74: now also JP3.2; no longer JP2.3
- net N$95: now also JP3.1; no longer JP2.4
- net N$96: now also JP3.3; no longer JP2.2
